Commit message: URDF update

File: urdf/yorat.urdf (robot description, URDF)
Before this commit: robot yorat, 4 links, 3 joints
Links:
- link base_link: mass 0.200 -> 0.500; geometry collision box size=0.07 0.07 0.04; visual box size=0.07 0.07 0.04
- link caster_wheel: mass 0.05 -> 0.3; geometry collision box size=0.005 0.07 0.01; visual box size=0.005 0.07 0.01
Joints:
- removed joint base_caster
- removed joint base_left
- removed joint base_right
- added joint base_caster_joint: type fixed, parent base_link, child caster_wheel, origin xyz=0.03 0 -0.025 rpy=0 0 0, axis 0 0 0
- added joint base_left_joint: type continuous, parent base_link, child left_wheel, origin xyz=-0.02 0.04 -0.01 rpy=1.57 0 0, axis 0 0 -1
- added joint base_right_joint: type continuous, parent base_link, child right_wheel, origin xyz=-0.02 -0.04 -0.01 rpy=1.57 0 0, axis 0 0 -1
